Commit message: Add kinect

File: autlab5/urdf/kinect.urdf.xacro (robot description, xacro)
@@ -1,9 +1,7 @@
 <?xml version="1.0"?>
 <robot name="sensor_kinect" xmlns:xacro="http://ros.org/wiki/xacro">
-  <!-- <xacro:property name="cam_px" value="-0.087" /> -->
-  <xacro:property name="cam_px" value="0.0" />
+  <xacro:property name="cam_px" value="-0.1" />
   <xacro:property name="cam_py" value="-0.0125" />
-  <!-- <xacro:property name="cam_pz" value="0.2870" /> -->
-  <xacro:property name="cam_pz" value="0.1370" />
+  <xacro:property name="cam_pz" value="0.2870" />
   <xacro:property name="cam_or" value="0" />
   <xacro:property name="cam_op" value="0" />
